File: fisk-batt-7.brd (EAGLE design)
At the start: 58.5 x 25.3 mm, 33 parts, among them IC3 MCP1703CB, U2 MCP73831T-2ACI/OT, X1 16 MHz

Commit message: update
Parts:
- renumbered U$2 to D1
Routing:
- net VBAT: track 36.2 -> 35.2 mm
Other:
- outline, holes or cut-outs redrawn
- board text added: "A0"
- board text added: "A1"
- board text added: "A2"
- board text added: "FSK"
- board text added: "VBAT"
- board text added: "VCC"
- board text added: "VIN"
