File: fisk-batt-7.sch (EAGLE design)
At the start: 33 parts, among them IC3 MCP1703CB, U2 MCP73831T-2ACI/OT, X1 16 MHz

Commit message: update
Parts:
- renumbered U$2 to D1
Changed lines of the file:
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@@
 <part name="C2" library="LowPowerLab" deviceset="CAP" device="0603-CAP" value="1u"/>
 <part name="C3" library="LowPowerLab" deviceset="CAP" device="0805-CAP" value="10u"/>
-<part name="U$2" library="LowPowerLab" deviceset="LED" device="0603"/>
+<part name="D1" library="LowPowerLab" deviceset="LED" device="0603"/>
 <part name="SUPPLY6" library="supply2" deviceset="GND" device=""/>
 <part name="R2" library="LowPowerLab" deviceset="RESISTOR" device="0603-RES" value="1k5"/>
@@
 <instance part="C2" gate="G$1" x="408.94" y="91.44"/>
 <instance part="C3" gate="G$1" x="365.76" y="91.44"/>
-<instance part="U$2" gate="G$1" x="102.87" y="73.66" smashed="yes" rot="R90"/>
+<instance part="D1" gate="G$1" x="102.87" y="73.66" smashed="yes" rot="R90"/>
 <instance part="SUPPLY6" gate="GND" x="102.87" y="66.04"/>
 <instance part="R2" gate="G$1" x="102.87" y="86.36" smashed="yes" rot="R90">
@@
 </segment>
 <segment>
-<pinref part="U$2" gate="G$1" pin="MINUS"/>
+<pinref part="D1" gate="G$1" pin="MINUS"/>
 <pinref part="SUPPLY6" gate="GND" pin="GND"/>
 <wire x1="102.87" y1="68.58" x2="102.87" y2="71.12" width="0.1524" layer="91"/>
@@
 <segment>
 <pinref part="R2" gate="G$1" pin="1"/>
-<pinref part="U$2" gate="G$1" pin="PLUS"/>
+<pinref part="D1" gate="G$1" pin="PLUS"/>
 <wire x1="102.87" y1="81.28" x2="102.87" y2="78.74" width="0.1524" layer="91"/>
 </segment>
@@
 <net name="VIN" class="0">
 <segment>
-<wire x1="388.62" y1="124.46" x2="408.94" y2="124.46" width="0.1524" layer="91"/>
+<wire x1="388.62" y1="124.46" x2="396.24" y2="109.22" width="0.1524" layer="91"/>
 <label x="406.4" y="127" size="1.778" layer="95"/>
 <wire x1="401.32" y1="96.52" x2="408.94" y2="96.52" width="0.1524" layer="91"/>
@@
 <label x="402.59" y="96.52" size="1.778" layer="95"/>
 <pinref part="C2" gate="G$1" pin="1"/>
-<wire x1="408.94" y1="124.46" x2="408.94" y2="96.52" width="0.1524" layer="91"/>
+<wire x1="396.24" y1="109.22" x2="408.94" y2="96.52" width="0.1524" layer="91"/>
 <pinref part="J10" gate="J$1" pin="2"/>
 <junction x="408.94" y="96.52"/>
